Commit message: Fix lidar near field and camera position

File: andino_webots/urdf/andino_webots_description.urdf.xacro (robot description, xacro)
@@ -1,4 +1,22 @@
 <?xml version="1.0"?>
 <robot xmlns:xacro="http://www.ros.org/wiki/xacro" name="andino">
+  <!--
+    In order for the generated proto to add Webots senors the origin urdf must contain gazebo-specific sensors.
+    The andino_gazebo xacro is used as base rather than the andino description to addresss this
+  -->
   <xacro:include filename="$(find andino_gazebo)/urdf/andino.gazebo.xacro"/>
+  <link name="webots_camera_link">
+    <visual>
+      <origin xyz="0 0 0" rpy="0 0 0"/>
+      <geometry>
+        <box size="0.001 0.001 0.001"/>
+      </geometry>
+    </visual>
+  </link>
+  <joint name="camera_rotation_joint" type="fixed">
+    <parent link="camera_link"/>
+    <child link="webots_camera_link"/>
+    <origin xyz="0 0 0" rpy="-1.5708 0 -1.5708"/>
+    <axis xyz="1 0 0" />
+  </joint>
 </robot>

Commit message: Revert "Fix lidar near field and camera position"
This reverts commit 5f9f3a7e9379a2f9e9d8d21b364da8abe3ab2b39.

File: andino_webots/urdf/andino_webots_description.urdf.xacro (robot description, xacro)
@@ -1,22 +1,4 @@
 <?xml version="1.0"?>
 <robot xmlns:xacro="http://www.ros.org/wiki/xacro" name="andino">
-  <!--
-    In order for the generated proto to add Webots senors the origin urdf must contain gazebo-specific sensors.
-    The andino_gazebo xacro is used as base rather than the andino description to addresss this
-  -->
   <xacro:include filename="$(find andino_gazebo)/urdf/andino.gazebo.xacro"/>
-  <link name="webots_camera_link">
-    <visual>
-      <origin xyz="0 0 0" rpy="0 0 0"/>
-      <geometry>
-        <box size="0.001 0.001 0.001"/>
-      </geometry>
-    </visual>
-  </link>
-  <joint name="camera_rotation_joint" type="fixed">
-    <parent link="camera_link"/>
-    <child link="webots_camera_link"/>
-    <origin xyz="0 0 0" rpy="-1.5708 0 -1.5708"/>
-    <axis xyz="1 0 0" />
-  </joint>
 </robot>

Commit message: Reformatted code
Signed-off-by: IDavGal <ignacio.davila@ekumenlabs.com>

File: andino_webots/urdf/andino_webots_description.urdf.xacro (robot description, xacro)
@@ -2,20 +2,21 @@
 <robot xmlns:xacro="http://www.ros.org/wiki/xacro" name="andino">
   <!--
-    In order for the generated proto to add Webots senors the origin urdf must contain gazebo-specific sensors.
+    In order for the generated proto to add Webots senors the origin urdf must contain gazebo-specific
+  sensors.
     The andino_gazebo xacro is used as base rather than the andino description to addresss this
   -->
-  <xacro:include filename="$(find andino_gazebo)/urdf/andino.gazebo.xacro"/>
+  <xacro:include filename="$(find andino_gazebo)/urdf/andino.gazebo.xacro" />
   <link name="webots_camera_link">
     <visual>
-      <origin xyz="0 0 0" rpy="0 0 0"/>
+      <origin xyz="0 0 0" rpy="0 0 0" />
       <geometry>
-        <box size="0.001 0.001 0.001"/>
+        <box size="0.001 0.001 0.001" />
       </geometry>
     </visual>
   </link>
   <joint name="camera_rotation_joint" type="fixed">
-    <parent link="camera_link"/>
-    <child link="webots_camera_link"/>
-    <origin xyz="0 0 0" rpy="-1.5708 0 -1.5708"/>
+    <parent link="camera_link" />
+    <child link="webots_camera_link" />
+    <origin xyz="0 0 0" rpy="-1.5708 0 -1.5708" />
     <axis xyz="1 0 0" />
   </joint>
